Commit message: mobile_robot_description: replace mesh collisions with primitive shapes
Swap chassis/wheels/lidar <collision> blocks from STL meshes to
<box>/<cylinder> primitives sized from each mesh's bounding box,
for faster and cleaner physics contacts. inspect_mesh.py also now
prints the bbox center and a ready-to-paste <collision> snippet,
so the URDF and the suggester stay in sync.

File: mobile_robot_description/urdf/mobile_robot.urdf.xacro (robot description, xacro)
@@ -29,8 +29,8 @@
       <material name="grayish-brown"></material>
     </visual>
-    <!-- Chassis Collision -->
+    <!-- Chassis Collision (bbox primitive, see scripts/inspect_mesh.py) -->
     <collision>
-      <origin xyz="0 0 0" rpy="0 0 0"/>
-      <geometry><mesh filename="file://$(find mobile_robot_description)/meshes/chassis.STL"/></geometry>
+      <origin xyz="0 0 0.6782" rpy="0 0 0"/>
+      <geometry><box size="0.6146 0.5660 1.3060"/></geometry>
     </collision>
   </link>
@@ -96,7 +96,8 @@
       <material name="black"></material>
     </visual>
+    <!-- Cylinder collision along Y (axle), see scripts/inspect_mesh.py -->
     <collision>
-      <origin xyz="0 0 0"/>
-      <geometry><mesh filename="file://$(find mobile_robot_description)/meshes/left_wheel_link.STL"/></geometry>
+      <origin xyz="0 -0.0205 0" rpy="1.5708 0 0"/>
+      <geometry><cylinder radius="0.0744" length="0.0410"/></geometry>
     </collision>
   </link>
@@ -123,7 +124,8 @@
       <material name="black"></material>
     </visual>
+    <!-- Cylinder collision along Y (axle), see scripts/inspect_mesh.py -->
     <collision>
-      <origin xyz="0 0 0"/>
-      <geometry><mesh filename="file://$(find mobile_robot_description)/meshes/right_wheel_link.STL"/></geometry>
+      <origin xyz="0 0.0165 0" rpy="1.5708 0 0"/>
+      <geometry><cylinder radius="0.0744" length="0.0410"/></geometry>
     </collision>
   </link>
@@ -160,7 +162,8 @@
       <material name="white"></material>
     </visual>
+    <!-- Cylinder collision along Z, see scripts/inspect_mesh.py -->
     <collision>
-      <origin xyz="0 0 0"/>
-      <geometry><mesh filename="file://$(find mobile_robot_description)/meshes/lidar.STL"/></geometry>
+      <origin xyz="-0.0227 0 -0.0069" rpy="0 0 0"/>
+      <geometry><cylinder radius="0.0303" length="0.0877"/></geometry>
     </collision>
   </link>

Commit message: perf(meshes): reduce face count on robot links via Blender Decimate
Apply Decimate modifier (Planar + Collapse) in Blender to optimize
STL mesh complexity for real-time simulation performance in Gazebo.

Affected links:
- chassis_link:     52,244 → 8,623 faces  (Planar 5° + Collapse 0.5)
- left_wheel_link:  3,570  → 1,784 faces  (Collapse 0.5)
- right_wheel_link: 3,570  → 1,784 faces  (Collapse 0.5)
- lidar_link:       8,152  → 982 faces    (Planar 5° + Collapse 0.15)

Collision meshes use primitive shapes in URDF are unaffected by this change.

File: mobile_robot_description/urdf/mobile_robot.urdf.xacro (robot description, xacro)
@@ -26,5 +26,5 @@
     <visual>
       <origin xyz="0 0 0" rpy="0 0 0"/>
-      <geometry><mesh filename="file://$(find mobile_robot_description)/meshes/chassis.STL"/></geometry>
+      <geometry><mesh filename="file://$(find mobile_robot_description)/meshes/chassis_link.STL"/></geometry>
       <material name="grayish-brown"></material>
     </visual>
@@ -159,5 +159,5 @@
     <visual>
       <origin xyz="0 0 0"/>
-      <geometry><mesh filename="file://$(find mobile_robot_description)/meshes/lidar.STL"/></geometry>
+      <geometry><mesh filename="file://$(find mobile_robot_description)/meshes/lidar_link.STL"/></geometry>
       <material name="white"></material>
     </visual>

Commit message: Normalize mesh file extensions to .stl and unify wheel meshes
- Renamed all mesh files from .STL to lowercase .stl
- Consolidated left/right wheel meshes into a single wheel_link.stl

File: mobile_robot_description/urdf/mobile_robot.urdf.xacro (robot description, xacro)
@@ -26,5 +26,5 @@
     <visual>
       <origin xyz="0 0 0" rpy="0 0 0"/>
-      <geometry><mesh filename="file://$(find mobile_robot_description)/meshes/chassis_link.STL"/></geometry>
+      <geometry><mesh filename="file://$(find mobile_robot_description)/meshes/chassis_link.stl"/></geometry>
       <material name="grayish-brown"></material>
     </visual>
@@ -93,5 +93,5 @@
     <visual>
       <origin xyz="0 0 0"/>
-      <geometry><mesh filename="file://$(find mobile_robot_description)/meshes/left_wheel_link.STL"/></geometry>
+      <geometry><mesh filename="file://$(find mobile_robot_description)/meshes/wheel_link.stl"/></geometry>
       <material name="black"></material>
     </visual>
@@ -121,5 +121,5 @@
     <visual>
       <origin xyz="0 0 0"/>
-      <geometry><mesh filename="file://$(find mobile_robot_description)/meshes/right_wheel_link.STL"/></geometry>
+      <geometry><mesh filename="file://$(find mobile_robot_description)/meshes/wheel_link.stl"/></geometry>
       <material name="black"></material>
     </visual>
@@ -159,5 +159,5 @@
     <visual>
       <origin xyz="0 0 0"/>
-      <geometry><mesh filename="file://$(find mobile_robot_description)/meshes/lidar_link.STL"/></geometry>
+      <geometry><mesh filename="file://$(find mobile_robot_description)/meshes/lidar_link.stl"/></geometry>
       <material name="white"></material>
     </visual>

Commit message: chore: change chassis link visualization to Orange

File: mobile_robot_description/urdf/mobile_robot.urdf.xacro (robot description, xacro)
@@ -27,5 +27,5 @@
       <origin xyz="0 0 0" rpy="0 0 0"/>
       <geometry><mesh filename="file://$(find mobile_robot_description)/meshes/chassis_link.stl"/></geometry>
-      <material name="grayish-brown"></material>
+      <material name="orange"></material>
     </visual>
     <!-- Chassis Collision (bbox primitive, see scripts/inspect_mesh.py) -->

Commit message: fix(description): mirror right wheel visual so it sits inboard
The shared wheel_link.stl is modeled asymmetrically about its
link origin (Y in [-0.041, 0]) — all geometry extends in -Y.

At the left wheel joint (y=+0.241) the mesh extends inboard
toward the chassis, which is correct. At the right wheel joint
(y=-0.241), the same unflipped mesh extends further outboard,
making the wheel appear stuck to the side of the chassis in
Gazebo instead of tucked under it.

Rotating the right wheel visual 180 deg about X
(rpy="3.14159 0 0") mirrors the mesh along Y so it extends
inboard, matching the left wheel. The collision cylinder offset
is also mirrored (-0.0205 -> +0.0205) so collision and visual
stay aligned.

File: mobile_robot_description/urdf/mobile_robot.urdf.xacro (robot description, xacro)
@@ -120,5 +120,6 @@
     </inertial>
     <visual>
-      <origin xyz="0 0 0"/>
+      <!-- Flip mesh along Y so the wheel sits inboard (mesh is modeled with Y in [-0.041, 0]) -->
+      <origin xyz="0 0 0" rpy="3.14159 0 0"/>
       <geometry><mesh filename="file://$(find mobile_robot_description)/meshes/wheel_link.stl"/></geometry>
       <material name="black"></material>
@@ -126,5 +127,5 @@
     <!-- Cylinder collision along Y (axle), see scripts/inspect_mesh.py -->
     <collision>
-      <origin xyz="0 0.0165 0" rpy="1.5708 0 0"/>
+      <origin xyz="0 0.0205 0" rpy="1.5708 0 0"/>
       <geometry><cylinder radius="0.0744" length="0.0410"/></geometry>
     </collision>
