Commit message: refactor(urdf): replace hardcoded radian literals with xacro pi constants
Swap ±1.570796 and 3.14 with ${pi/2}, ${-pi/2}, and ${pi} throughout
the description link, consistent with the pi convention already used
for wheel visuals and collision rotations. No numerical change.

File: mobile_robot_description/urdf/mobile_robot.gazebo.xacro (robot description, xacro)
@@ -118,6 +118,6 @@
             <samples>181</samples>
             <resolution>1</resolution>
-            <min_angle>-1.570796</min_angle>
-            <max_angle>1.570796</max_angle>
+            <min_angle>${-pi/2}</min_angle>
+            <max_angle>${pi/2}</max_angle>
           </horizontal>
         </scan>

File: mobile_robot_description/urdf/mobile_robot.urdf.xacro (robot description, xacro)
@@ -98,5 +98,5 @@
     <!-- Cylinder collision along Y (axle), see scripts/inspect_mesh.py -->
     <collision>
-      <origin xyz="0 -0.0205 0" rpy="1.5708 0 0"/>
+      <origin xyz="0 -0.0205 0" rpy="${pi/2} 0 0"/>
       <geometry><cylinder radius="0.0744" length="0.0410"/></geometry>
     </collision>
@@ -121,5 +121,5 @@
     <visual>
       <!-- Flip mesh along Y so the wheel sits inboard (mesh is modeled with Y in [-0.041, 0]) -->
-      <origin xyz="0 0 0" rpy="3.14159 0 0"/>
+      <origin xyz="0 0 0" rpy="${pi} 0 0"/>
       <geometry><mesh filename="file://$(find mobile_robot_description)/meshes/wheel_link.stl"/></geometry>
       <material name="black"></material>
@@ -127,5 +127,5 @@
     <!-- Cylinder collision along Y (axle), see scripts/inspect_mesh.py -->
     <collision>
-      <origin xyz="0 0.0205 0" rpy="1.5708 0 0"/>
+      <origin xyz="0 0.0205 0" rpy="${pi/2} 0 0"/>
       <geometry><cylinder radius="0.0744" length="0.0410"/></geometry>
     </collision>
