Commit message: refactor(description): split robot models into Rooster and YuHou variants
Mirrors TurtleBot's Burger/Waffle pattern. The complex STL-based robot is
named Rooster; the simple parametric primitive-based robot (ported from
Differential-Drive-Mobile-Robot repo) is named YuHou.

- urdf/rooster/  — rooster.urdf.xacro, rooster.gazebo.xacro, materials.xacro
- urdf/yuhou/   — yuhou.urdf.xacro, yuhou.gazebo.xacro, inertia_macros.xacro
- meshes/rooster/ — STL files relocated from meshes/
- config/yuhou/  — robot_dimensions_config.yaml (YuHou parametric dims)
- Update all launch files and genesis scripts to point at rooster paths
- Update robot_dimensions_config_editor.py to point at yuhou config

File: mobile_robot_description/urdf/rooster/rooster.urdf.xacro (robot description, xacro)
@@ -1,7 +1,7 @@
 <?xml version='1.0'?>
-<robot name="mobile_robot_description" xmlns:xacro="http://www.ros.org/wiki/xacro">
+<robot name="rooster" xmlns:xacro="http://www.ros.org/wiki/xacro">
   <!-- ================== Includes ================== -->
-  <xacro:include filename="$(find mobile_robot_description)/urdf/mobile_robot.gazebo.xacro" />
-  <xacro:include filename="$(find mobile_robot_description)/urdf/materials.xacro" />
+  <xacro:include filename="$(find mobile_robot_description)/urdf/rooster/rooster.gazebo.xacro" />
+  <xacro:include filename="$(find mobile_robot_description)/urdf/rooster/materials.xacro" />
   <!--
     Robot Structure Overview:
@@ -26,5 +26,5 @@
     <visual>
       <origin xyz="0 0 0" rpy="0 0 0"/>
-      <geometry><mesh filename="file://$(find mobile_robot_description)/meshes/chassis_link.stl"/></geometry>
+      <geometry><mesh filename="file://$(find mobile_robot_description)/meshes/rooster/chassis_link.stl"/></geometry>
       <material name="orange"></material>
     </visual>
@@ -93,5 +93,5 @@
     <visual>
       <origin xyz="0 0 0"/>
-      <geometry><mesh filename="file://$(find mobile_robot_description)/meshes/wheel_link.stl"/></geometry>
+      <geometry><mesh filename="file://$(find mobile_robot_description)/meshes/rooster/wheel_link.stl"/></geometry>
       <material name="black"></material>
     </visual>
@@ -122,5 +122,5 @@
       <!-- Flip mesh along Y so the wheel sits inboard (mesh is modeled with Y in [-0.041, 0]) -->
       <origin xyz="0 0 0" rpy="${pi} 0 0"/>
-      <geometry><mesh filename="file://$(find mobile_robot_description)/meshes/wheel_link.stl"/></geometry>
+      <geometry><mesh filename="file://$(find mobile_robot_description)/meshes/rooster/wheel_link.stl"/></geometry>
       <material name="black"></material>
     </visual>
@@ -160,5 +160,5 @@
     <visual>
       <origin xyz="0 0 0"/>
-      <geometry><mesh filename="file://$(find mobile_robot_description)/meshes/lidar_link.stl"/></geometry>
+      <geometry><mesh filename="file://$(find mobile_robot_description)/meshes/rooster/lidar_link.stl"/></geometry>
       <material name="white"></material>
     </visual>
