Commit message: refactor(description): restructure into models/rooster and models/yuhou
Reorganize mobile_robot_description to per-robot subdirectories nested under models/:
models/rooster/{meshes,urdf} and models/yuhou/{config,urdf}.

Update all xacro includes, mesh paths, CMakeLists install target, config
editor script, launch files, and genesis scripts to match.

File: mobile_robot_description/models/rooster/urdf/rooster.urdf.xacro (robot description, xacro)
@@ -2,6 +2,6 @@
 <robot name="rooster" xmlns:xacro="http://www.ros.org/wiki/xacro">
   <!-- ================== Includes ================== -->
-  <xacro:include filename="$(find mobile_robot_description)/urdf/rooster/rooster.gazebo.xacro" />
-  <xacro:include filename="$(find mobile_robot_description)/urdf/rooster/materials.xacro" />
+  <xacro:include filename="$(find mobile_robot_description)/models/rooster/urdf/rooster.gazebo.xacro" />
+  <xacro:include filename="$(find mobile_robot_description)/models/rooster/urdf/materials.xacro" />
   <!--
     Robot Structure Overview:
@@ -26,5 +26,5 @@
     <visual>
       <origin xyz="0 0 0" rpy="0 0 0"/>
-      <geometry><mesh filename="file://$(find mobile_robot_description)/meshes/rooster/chassis_link.stl"/></geometry>
+      <geometry><mesh filename="file://$(find mobile_robot_description)/models/rooster/meshes/chassis_link.stl"/></geometry>
       <material name="orange"></material>
     </visual>
@@ -93,5 +93,5 @@
     <visual>
       <origin xyz="0 0 0"/>
-      <geometry><mesh filename="file://$(find mobile_robot_description)/meshes/rooster/wheel_link.stl"/></geometry>
+      <geometry><mesh filename="file://$(find mobile_robot_description)/models/rooster/meshes/wheel_link.stl"/></geometry>
       <material name="black"></material>
     </visual>
@@ -122,5 +122,5 @@
       <!-- Flip mesh along Y so the wheel sits inboard (mesh is modeled with Y in [-0.041, 0]) -->
       <origin xyz="0 0 0" rpy="${pi} 0 0"/>
-      <geometry><mesh filename="file://$(find mobile_robot_description)/meshes/rooster/wheel_link.stl"/></geometry>
+      <geometry><mesh filename="file://$(find mobile_robot_description)/models/rooster/meshes/wheel_link.stl"/></geometry>
       <material name="black"></material>
     </visual>
@@ -160,5 +160,5 @@
     <visual>
       <origin xyz="0 0 0"/>
-      <geometry><mesh filename="file://$(find mobile_robot_description)/meshes/rooster/lidar_link.stl"/></geometry>
+      <geometry><mesh filename="file://$(find mobile_robot_description)/models/rooster/meshes/lidar_link.stl"/></geometry>
       <material name="white"></material>
     </visual>

File: mobile_robot_description/models/yuhou/urdf/yuhou.urdf.xacro (robot description, xacro)
@@ -1,6 +1,6 @@
 <?xml version="1.0"?>
 <robot name="yuhou" xmlns:xacro="http://www.ros.org/wiki/xacro">
-  <xacro:include filename="$(find mobile_robot_description)/urdf/yuhou/inertia_macros.xacro"/>
-  <xacro:include filename="$(find mobile_robot_description)/urdf/yuhou/yuhou.gazebo.xacro"/>
+  <xacro:include filename="$(find mobile_robot_description)/models/yuhou/urdf/inertia_macros.xacro"/>
+  <xacro:include filename="$(find mobile_robot_description)/models/yuhou/urdf/yuhou.gazebo.xacro"/>
   <!-- robot_dimensions_config.yaml -->
   <xacro:property name="base_length" value="$(arg base_length)" />
